File: kicad/hux.kicad_pcb (KiCad board)
At the start: 2 copper layers, 72 x 72 mm, 21 parts, among them J1 USB-C-16P, J2 ST7789_1.69_IPS, J3 SPK_OUT, SW1 RST, SW2 BOOT, U1 ESP32-S3-WROOM-1, U3 TLV75533, U4 INMP441, U5 MAX98357A

Commit message: Add bill of materials and hardware specifications
Other:
- board text added: "SMART HOME COMPANION"
- board text removed: "STARK // JARVIS COMPANION"
Changed lines of the file:
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@@
 	(paper "A4")
 	(title_block
-		(title "Hux: Desktop AI Smart Home Assistant (Jarvis Companion)")
+		(title "Hux: Desktop AI Smart Home Assistant")
 		(date "2026-10-28")
 		(rev "v1.0")
@@
 	(gr_circle (center 36.0 34.0) (end 58.5 34.0) (stroke (width 0.2) (type default)) (layer "F.SilkS"))
 	(gr_text "HUX // AI DESKTOP ASSISTANT" (at 36.0 63.5) (layer "F.SilkS") (effects (font (size 1.3 1.3) (thickness 0.22) bold)))
-	(gr_text "STARK // JARVIS COMPANION" (at 36.0 66.5) (layer "F.SilkS") (effects (font (size 0.9 0.9) (thickness 0.18))))
+	(gr_text "SMART HOME COMPANION" (at 36.0 66.5) (layer "F.SilkS") (effects (font (size 0.9 0.9) (thickness 0.18))))
 	(gr_text "Hack Club Half Life // AwesomeSno" (at 36.0 69.2) (layer "F.SilkS") (effects (font (size 0.8 0.8) (thickness 0.16))))
 	(gr_text "MIC IN" (at 36.0 11.5) (layer "F.SilkS") (effects (font (size 0.8 0.8) (thickness 0.16))))
