File: kicad/hux.kicad_sch (KiCad schematic)
At the start: 19 parts, among them J1 TYPE-C-16P, J2 ST7789_1.69_IPS, J3 SPK_OUT, J4 I2C_EXT, SW1 RESET, SW2 BOOT, U1 ESP32-S3-WROOM-1, U2 USBLC6-2SC6, U3 TLV75533PDBVR, U4 INMP441, U5 MAX98357A

Commit message: Add bill of materials and hardware specifications
Other:
- title: Hux: Desktop AI Smart Home Assistant (Jarvis Companion) -> Hux: Desktop AI Smart Home Assistant
Changed lines of the file:
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@@
 	(paper "A3")
 	(title_block
-		(title "Hux: Desktop AI Smart Home Assistant (Jarvis Companion)")
+		(title "Hux: Desktop AI Smart Home Assistant")
 		(date "2026-10-28")
 		(rev "v1.0")
@@
 		(instances
 			(project "hux"
-				(path "/fef6db75-802f-4b68-806d-a4530399060a"
+				(path "/b6a3e7aa-1668-494e-bd37-1c1ad7485d0f"
 					(reference "U1")
 					(unit 1)
@@
 		(instances
 			(project "hux"
-				(path "/fef6db75-802f-4b68-806d-a4530399060a"
+				(path "/b6a3e7aa-1668-494e-bd37-1c1ad7485d0f"
 					(reference "J1")
 					(unit 1)
@@
 		(instances
 			(project "hux"
-				(path "/fef6db75-802f-4b68-806d-a4530399060a"
+				(path "/b6a3e7aa-1668-494e-bd37-1c1ad7485d0f"
 					(reference "U2")
 					(unit 1)
@@
 		(instances
 			(project "hux"
-				(path "/fef6db75-802f-4b68-806d-a4530399060a"
+				(path "/b6a3e7aa-1668-494e-bd37-1c1ad7485d0f"
 					(reference "U3")
 					(unit 1)
@@
 		(instances
 			(project "hux"
-				(path "/fef6db75-802f-4b68-806d-a4530399060a"
+				(path "/b6a3e7aa-1668-494e-bd37-1c1ad7485d0f"
 					(reference "J2")
 					(unit 1)
@@
 		(instances
 			(project "hux"
-				(path "/fef6db75-802f-4b68-806d-a4530399060a"
+				(path "/b6a3e7aa-1668-494e-bd37-1c1ad7485d0f"
 					(reference "U4")
 					(unit 1)
@@
 		(instances
 			(project "hux"
-				(path "/fef6db75-802f-4b68-806d-a4530399060a"
+				(path "/b6a3e7aa-1668-494e-bd37-1c1ad7485d0f"
 					(reference "U5")
 					(unit 1)
@@
 		(instances
 			(project "hux"
-				(path "/fef6db75-802f-4b68-806d-a4530399060a"
+				(path "/b6a3e7aa-1668-494e-bd37-1c1ad7485d0f"
 					(reference "J3")
 					(unit 1)
@@
 		(instances
 			(project "hux"
-				(path "/fef6db75-802f-4b68-806d-a4530399060a"
+				(path "/b6a3e7aa-1668-494e-bd37-1c1ad7485d0f"
 					(reference "J4")
 					(unit 1)
@@
 		(instances
 			(project "hux"
-				(path "/fef6db75-802f-4b68-806d-a4530399060a"
+				(path "/b6a3e7aa-1668-494e-bd37-1c1ad7485d0f"
 					(reference "SW1")
 					(unit 1)
@@
 		(instances
 			(project "hux"
-				(path "/fef6db75-802f-4b68-806d-a4530399060a"
+				(path "/b6a3e7aa-1668-494e-bd37-1c1ad7485d0f"
 					(reference "SW2")
 					(unit 1)
@@
 		(instances
 			(project "hux"
-				(path "/fef6db75-802f-4b68-806d-a4530399060a"
+				(path "/b6a3e7aa-1668-494e-bd37-1c1ad7485d0f"
 					(reference "LED1")
 					(unit 1)
@@
 		(instances
 			(project "hux"
-				(path "/fef6db75-802f-4b68-806d-a4530399060a"
+				(path "/b6a3e7aa-1668-494e-bd37-1c1ad7485d0f"
 					(reference "LED2")
 					(unit 1)
@@
 		(instances
 			(project "hux"
-				(path "/fef6db75-802f-4b68-806d-a4530399060a"
+				(path "/b6a3e7aa-1668-494e-bd37-1c1ad7485d0f"
 					(reference "LED3")
 					(unit 1)
@@
 		(instances
 			(project "hux"
-				(path "/fef6db75-802f-4b68-806d-a4530399060a"
+				(path "/b6a3e7aa-1668-494e-bd37-1c1ad7485d0f"
 					(reference "LED4")
 					(unit 1)
@@
 		(instances
 			(project "hux"
-				(path "/fef6db75-802f-4b68-806d-a4530399060a"
+				(path "/b6a3e7aa-1668-494e-bd37-1c1ad7485d0f"
 					(reference "LED5")
 					(unit 1)
@@
 		(instances
 			(project "hux"
-				(path "/fef6db75-802f-4b68-806d-a4530399060a"
+				(path "/b6a3e7aa-1668-494e-bd37-1c1ad7485d0f"
 					(reference "LED6")
 					(unit 1)
@@
 		(instances
 			(project "hux"
-				(path "/fef6db75-802f-4b68-806d-a4530399060a"
+				(path "/b6a3e7aa-1668-494e-bd37-1c1ad7485d0f"
 					(reference "LED7")
 					(unit 1)
@@
 		(instances
 			(project "hux"
-				(path "/fef6db75-802f-4b68-806d-a4530399060a"
+				(path "/b6a3e7aa-1668-494e-bd37-1c1ad7485d0f"
 					(reference "LED8")
 					(unit 1)
